Commit message: feat: launched simulation

File: src/assets/urdf/jettank.urdf (robot description, URDF)
Before this commit: robot jettank, 9 links, 8 joints
Links:
- link back_shell_link: geometry collision mesh filename=package://tank_description/meshes/back_shell_link.stl; visual mesh filename=package://tank_description/meshes/back_shell_link.stl
- link base_link: geometry collision box size=0.297 0.145 0.11255; visual mesh filename=package://tank_description/meshes/base_link.stl
- link camera_link: geometry collision mesh filename=package://tank_description/meshes/depth_camera_link.stl; visual mesh filename=package://tank_description/meshes/depth_camera_link.stl
- link lidar_link: geometry collision mesh filename=package://tank_description/meshes/lidar_link.stl; visual mesh filename=package://tank_description/meshes/lidar_link.stl
- link wheel_link: geometry collision mesh filename=package://tank_description/meshes/wheel.stl; visual mesh filename=package://tank_description/meshes/wheel.stl
