Commit message: feat: first simple training

File: projects/pirl/source/pirl/pirl/assets/urdf/jettank.urdf (robot description, URDF)
Before this commit: robot jettank, 9 links, 8 joints
Links:
- removed link back_shell_link
- removed link camera_frame
- removed link imu_link
- removed link lidar_frame
- removed link wheel_link
- added link left_wheel, mass 0.1; collision cylinder length=0.04 radius=0.05; visual cylinder length=0.04 radius=0.05
- added link right_wheel, mass 0.1; collision cylinder length=0.04 radius=0.05; visual cylinder length=0.04 radius=0.05
- link base_link: geometry collision box size=0.297 0.145 0.11255; visual box size=0.297 0.145 0.11255
- link camera_link: mass 0.227980406655671 -> None; geometry visual box size=0.02 0.05 0.02
- link lidar_link: mass 0.0522535578752524 -> None; geometry visual cylinder length=0.03 radius=0.03
Joints:
- removed joint back_shell_joint
- removed joint camera_joint_sim
- removed joint imu_joint
- removed joint joint1
- removed joint lidar_frame_joint
- removed joint wheel_joint
- added joint camera_joint: type fixed, parent base_link, child camera_link, origin xyz=0.14 0 0.05 rpy=0 0 0
- added joint left_wheel_joint: type continuous, parent base_link, child left_wheel, origin xyz=0.1 0.08 -0.025 rpy=0 0 0, axis 0 1 0
- added joint right_wheel_joint: type continuous, parent base_link, child right_wheel, origin xyz=0.1 -0.08 -0.025 rpy=0 0 0, axis 0 1 0
- joint base_joint: origin xyz=0.0 0.0 0.0 rpy=0 0 0 -> xyz=0.0 0.0 0.05 rpy=0 0 0
- joint lidar_joint: axis 0 0 0 -> (none); origin xyz=0.0959394346777203 -1.03974386779226E-05 0.128396206697751 rpy=0 0 0 -> xyz=0.1 0 0.1 rpy=0 0 0

Commit message: feat: added inflation layer in costmap & missing meshes

File: projects/pirl/source/pirl/pirl/assets/urdf/jettank.urdf (robot description, URDF)
Before this commit: robot jettank, 6 links, 5 joints
Links:
- added link back_shell_link, mass 0.0663479; collision mesh filename=../meshes/back_shell_link.stl; visual mesh filename=../meshes/back_shell_link.stl
- added link front_skid; collision box size=0.10 0.10 0.02
- added link left_roller_rear, mass 0.05; visual cylinder length=0.04 radius=0.03
- added link right_roller_rear, mass 0.05; visual cylinder length=0.04 radius=0.03
- added link track_visual; visual mesh filename=../meshes/wheel.stl
- link base_link: geometry collision box size=0.297 0.145 0.11255; visual mesh filename=../meshes/base_link.stl
- link camera_link: mass None -> 0.2279804; geometry collision mesh filename=../meshes/depth_camera_link.stl; visual mesh filename=../meshes/depth_camera_link.stl
- link lidar_link: mass None -> 0.0522536; geometry collision mesh filename=../meshes/lidar_link.stl; visual mesh filename=../meshes/lidar_link.stl
Joints:
- added joint back_shell_joint: type fixed, parent base_link, child back_shell_link, origin xyz=-0.076481 0 0.082796 rpy=-3.1416 0 1.5708, axis 0 0 0
- added joint front_skid_joint: type fixed, parent base_link, child front_skid, origin xyz=0 0 0 rpy=0 0 0, axis 0 0 0
- added joint left_roller_rear_joint: type continuous, parent base_link, child left_roller_rear, origin xyz=-0.14 0.08 -0.03 rpy=0 0 0, axis 0 1 0
- added joint right_roller_rear_joint: type continuous, parent base_link, child right_roller_rear, origin xyz=-0.14 -0.08 -0.03 rpy=0 0 0, axis 0 1 0
- added joint track_visual_joint: type fixed, parent base_link, child track_visual, origin xyz=0 0 0 rpy=0 0 0, axis 0 0 0
- joint base_joint: origin xyz=0.0 0.0 0.05 rpy=0 0 0 -> xyz=0.0 0.0 0.0 rpy=0 0 0
- joint camera_joint: axis (none) -> 0 0 0; origin xyz=0.14 0 0.05 rpy=0 0 0 -> xyz=0.0288581 0 0.2020933 rpy=-0.0001315 0 0
- joint left_wheel_joint: origin xyz=0.1 0.08 -0.025 rpy=0 0 0 -> xyz=-0.06 0.08 -0.02 rpy=0 0 0
- joint lidar_joint: axis (none) -> 0 0 0; origin xyz=0.1 0 0.1 rpy=0 0 0 -> xyz=0.0959394 -0.0000104 0.1283962 rpy=0 0 0
- joint right_wheel_joint: origin xyz=0.1 -0.08 -0.025 rpy=0 0 0 -> xyz=-0.06 -0.08 -0.02 rpy=0 0 0

Commit message: fix(urdf): fixed robot meshes by removing handmade prims

File: projects/pirl/source/pirl/pirl/assets/urdf/jettank.urdf (robot description, URDF)
Before this commit: robot jettank, 11 links, 10 joints
Links:
- removed link left_roller_rear
- removed link right_roller_rear
- link left_wheel: geometry collision cylinder length=0.04 radius=0.03
- link right_wheel: geometry collision cylinder length=0.04 radius=0.03
Joints:
- removed joint left_roller_rear_joint
- removed joint right_roller_rear_joint
- joint left_wheel_joint: origin xyz=-0.06 0.08 -0.02 rpy=0 0 0 -> xyz=-0.06 0.121 0.01 rpy=0 0 0
- joint right_wheel_joint: origin xyz=-0.06 -0.08 -0.02 rpy=0 0 0 -> xyz=-0.06 -0.121 0.01 rpy=0 0 0

Commit message: refactor: seperated proximity & move obstacles logic from pirl_env.py

File: projects/pirl/source/pirl/pirl/assets/urdf/jettank.urdf (robot description, URDF)
Before this commit: robot jettank, 9 links, 8 joints
Joints:
- joint back_shell_joint: origin xyz=-0.076481 0 0.082796 rpy=-3.1416 0 1.5708 -> xyz=-0.076481 0.0 0.082796 rpy=-3.1416 0 1.5708
- joint camera_joint: origin xyz=0.0288581 0 0.2020933 rpy=-0.0001315 0 0 -> xyz=0.0288581 0.0 0.2020933 rpy=-0.0001315 0 0
- joint lidar_joint: origin xyz=0.0959394 -0.0000104 0.1283962 rpy=0 0 0 -> xyz=0.0959394 0.0 0.1283962 rpy=0 0 0

Commit message: fix(lidar): changed lidar pitch to neutral

File: projects/pirl/source/pirl/pirl/assets/urdf/jettank.urdf (robot description, URDF)
Before this commit: robot jettank, 9 links, 8 joints
Joints:
- joint lidar_joint: origin xyz=0.0959394 0.0 0.1283962 rpy=0 0 0 -> xyz=0.0959394 0.0 0.1283962 rpy=0 -0.0436332313 0
